File: Macropad.kicad_sch (KiCad schematic)
At the start: 4 parts, among them J1 USB_C_Receptacle_USB2.0_16P, U1 ATmega32U4-M, Y1 Resonator

Commit message: component layout
Parts:
- removed Y1: Resonator, symbol Device:Resonator
- added C1, C2: 22p, Capacitor_SMD:C_0201_0603Metric_Pad0.64x0.40mm_HandSolder, symbol Device:C
- added C3: 1u, Capacitor_SMD:C_0201_0603Metric_Pad0.64x0.40mm_HandSolder, symbol Device:C
- added D1, D2, D3, D4: LED, LED_THT:LED_D1.8mm_W3.3mm_H2.4mm, symbol Device:LED
- added F1: 500mA, Fuse:Fuse_0603_1608Metric, symbol Device:Fuse
- added J2: AVR-ISP-6, Connector_IDC:IDC-Header_2x03_P2.54mm_Vertical_SMD, symbol Connector:AVR-ISP-6
- added Mode_SW1: SW_Push, Button_Switch_THT:SW_PUSH-12mm, symbol Switch:SW_Push
- added R1, R6: 10k, PCM_Resistor_THT_AKL:R_Axial_DIN0204_L3.6mm_D1.6mm_P5.08mm_Horizontal, symbol Device:R
- added R2, R3: 22, PCM_Resistor_THT_AKL:R_Axial_DIN0204_L3.6mm_D1.6mm_P5.08mm_Horizontal, symbol Device:R
- added R4, R5: 5k1, PCM_Resistor_THT_AKL:R_Axial_DIN0204_L3.6mm_D1.6mm_P5.08mm_Horizontal, symbol Device:R
- added ROTARY_SW1, ROTARY_SW2: RotaryEncoder_Switch_MP, Rotary_Encoder:RotaryEncoder_Alps_EC12E-Switch_Vertical_H20mm, symbol Device:RotaryEncoder_Switch_MP
- added SW1, SW10, SW2, SW3, SW4, SW5, SW6, SW7, SW8, SW9: SW_Push, PCM_Switch_Keyboard_Cherry_MX:SW_Cherry_MX_PCB, symbol Switch:SW_Push
- added Y1: Crystal_GND2, Crystal:Resonator-3Pin_W7.0mm_H2.5mm, symbol Device:Crystal_GND2
- J1: footprint (none) -> Connector_USB:USB_C_Receptacle_GCT_USB4105-xx-A_16P_TopMnt_Horizontal
- Reset_SW1: renamed from Reset_SW; footprint (none) -> Button_Switch_THT:SW_PUSH_6mm
Connections:
- net at U1.10 (PB2): now also J2.4 (MOSI)
- net at U1.11 (PB3): now also J2.1 (MISO)
- net at U1.13 (~{RESET}): now also Reset_SW1.2, J2.5 (~{RST}), R1.2
- net at U1.16 (XTAL2): now also C2.1, Y1.1
- net at U1.17 (XTAL1): now also C1.1, Y1.3
- net at U1.3 (D-): now also R2.2
- net at U1.33 (~{HWB}/PE2): now also R6.1
- net at U1.4 (D+): now also R3.2
- net at U1.6 (UCAP): now also C3.1
- net at U1.7 (VBUS): now also F1.2
- net at U1.9 (PB1): now also J2.3 (SCK)
- net at J1.A4 (VBUS), J1.A9 (VBUS), J1.B4 (VBUS)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: now also F1.1
- net at J1.A5 (CC1): now also R4.1
- net at J1.A6 (D+): now also J1.B6 (D+), R3.1
- net at J1.A7 (D-): now also J1.B7 (D-), R2.1
- net at J1.B5 (CC2): now also R5.1
- new net: C1.2, C2.2, Y1.2
- no-connect marks 0 -> 3
Other:
- moved on the sheet: J1, Reset_SW1, U1
